File: PCB_CNC_Prototype/Solenoid_Array_CNCPrototype.sch (KiCad schematic (older format))
At the start: 20 parts, among them J1 Conn_01x02, J16 Power Daisy Chain_input, J17 Power Daisy Chain_Output, J2 Conn_01x02, J3 Conn_01x01, J4 Conn_01x01, Q1 AOD508, Q2 AOD508

Commit message: Add files via upload
Parts:
- removed C2: EMK325ABJ107MM-T, troglodisme_footprints:CAPC3225X270N, symbol troglodisme_symbols:EMK325ABJ107MM-T
- removed D17: IN-S126AT5UW, troglodisme_footprints:IN-S126AT5UW, symbol troglodisme_symbols:IN-S126AT5UW
- removed D2: SD1206S040S2R0, troglodisme_footprints:SD1206S040S2R0, symbol troglodisme_symbols:SD1206S040S2R0
- removed J17: Power Daisy Chain_Output, troglodisme_footprints:JST_PH_S2B-PH-K_1x02_P2.00mm_Horizontal_noSilkScreen, symbol Connector_Generic:Conn_01x02
- removed J2: Conn_01x02, troglodisme_footprints:JST_PH_S2B-PH-K_1x02_P2.00mm_Horizontal_noSilkScreen, symbol Connector_Generic:Conn_01x02
- removed J4: Conn_01x01, Connector_PinHeader_2.54mm:PinHeader_1x01_P2.54mm_Vertical, symbol Connector_Generic:Conn_01x01
- removed Q2: AOD508, troglodisme_footprints:AOD508, symbol troglodisme_symbols:AOD508
- removed R18: 100K, Resistor_SMD:R_1210_3225Metric_Pad1.42x2.65mm_HandSolder, symbol Device:R
- removed R2: 150R, Resistor_SMD:R_1210_3225Metric_Pad1.42x2.65mm_HandSolder, symbol Device:R
- removed R33: 470R, Resistor_SMD:R_1210_3225Metric_Pad1.42x2.65mm_HandSolder, symbol Device:R
- C1: symbol troglodisme_symbols:EMK325ABJ107MM-T -> Solenoid_Array_CNCPrototype-rescue:EMK325ABJ107MM-T-troglodisme_symbols
- D1: symbol troglodisme_symbols:SD1206S040S2R0 -> Solenoid_Array_CNCPrototype-rescue:SD1206S040S2R0-troglodisme_symbols
- D16: symbol troglodisme_symbols:IN-S126AT5UW -> Solenoid_Array_CNCPrototype-rescue:IN-S126AT5UW-troglodisme_symbols
- Q1: symbol troglodisme_symbols:AOD508 -> Solenoid_Array_CNCPrototype-rescue:AOD508-troglodisme_symbols
Connections:
- wire segments 62 -> 35
