File: PCB_CNC_Prototype/Solenoid_Array_CNCPrototype.kicad_pcb (KiCad board)
At the start: 2 copper layers, 767.7 x 345.5 mm, 10 parts, among them J1 Conn_01x02, J16 Power Daisy Chain_input, J3 Conn_01x01, Q1 AOD508

Commit message: .
Parts:
- moved C1 2.54 mm to (102.4, 179.0)
Routing:
- net +5V: track 0.00 -> 53.3 mm
- net Net-(D1-Pad2): track 0.00 -> 43.4 mm
- net GND: track 0.00 -> 20.3 mm
- net Net-(D16-Pad2): track 0.00 -> 10.2 mm
- net Net-(J3-Pad1): track 13.3 -> 14.8 mm
Changed lines of the file:
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@@
     (thickness 1.6002)
     (drawings 14)
-    (tracks 8)
+    (tracks 36)
     (zones 0)
     (modules 10)
@@
   )
   (setup
-    (last_trace_width 0.25)
+    (last_trace_width 1)
     (user_trace_width 0.1)
     (user_trace_width 0.2)
@@
   )
   (module troglodisme_footprints:CAPC3225X270N (layer Front)
-    (at 102.875 176.5)
+    (at 102.4 179)
     (descr EMK325ABJ107MM-T-1)
     (tags "Capacitor 1206")
@@
   (gr_circle (center 127 172) (end 128.5 172) (layer Edge.Cuts) (width 0.1))
   (gr_circle (center 87 199) (end 88.5 199) (layer Edge.Cuts) (width 0.1))
-  (gr_text "VCC+\n" (at 87.54 179.43 90) (layer Front)
+  (gr_text "VCC+\n" (at 103.66 187.45 180) (layer Front)
     (effects (font (size 1.5 1.5) (thickness 0.3)))
   )
@@
   (gr_curve (pts (xy 850.695064 -142.464645) (xy 850.695064 -142.464645) (xy 849.695064 -142.464645) (xy 849.695064 -142.464645)) (layer Edge.Cuts) (width 0.2))
   (gr_curve (pts (xy 849.695064 -142.464645) (xy 849.695064 -142.464645) (xy 850.695064 -142.464645) (xy 850.695064 -142.464645)) (layer Edge.Cuts) (width 0.2))
-  (segment (start 117.146 184.2915) (end 117.54 183.8975) (width 0.25) (layer Front) (net 4))
-  (segment (start 117.146 190.32) (end 117.146 184.2915) (width 0.25) (layer Front) (net 4))
-  (segment (start 113.47 176.81) (end 111.97 176.81) (width 0.25) (layer Front) (net 6))
-  (segment (start 117.54 180.21) (end 114.14 176.81) (width 0.25) (layer Front) (net 6))
-  (segment (start 114.14 176.81) (end 113.47 176.81) (width 0.25) (layer Front) (net 6))
-  (segment (start 117.54 180.9225) (end 117.54 180.21) (width 0.25) (layer Front) (net 6))
-  (segment (start 117.49 180.8725) (end 117.54 180.9225) (width 0.25) (layer Front) (net 6))
-  (segment (start 111.95 180.8725) (end 117.49 180.8725) (width 0.25) (layer Front) (net 6))
+  (segment (start 101.46 183.96) (end 98.02 183.96) (width 1) (layer Front) (net 1))
+  (segment (start 96.08 185.9) (end 96.08 188.65) (width 1) (layer Front) (net 1))
+  (segment (start 98.02 183.96) (end 96.08 185.9) (width 1) (layer Front) (net 1))
+  (segment (start 101.05 183.55) (end 101.46 183.96) (width 1) (layer Front) (net 1))
+  (segment (start 101.05 179) (end 101.05 183.55) (width 1) (layer Front) (net 1))
+  (segment (start 124.46 180.7825) (end 115.3375 171.66) (width 1) (layer Front) (net 1))
+  (segment (start 106.03 171.66) (end 101.05 176.64) (width 1) (layer Front) (net 1))
+  (segment (start 101.05 176.64) (end 101.05 179) (width 1) (layer Front) (net 1))
+  (segment (start 115.3375 171.66) (end 106.03 171.66) (width 1) (layer Front) (net 1))
+  (segment (start 94.58 179.26) (end 93.08 179.26) (width 1) (layer Front) (net 1))
+  (segment (start 98.02 182.7) (end 94.58 179.26) (width 1) (layer Front) (net 1))
+  (segment (start 98.02 183.96) (end 98.02 182.7) (width 1) (layer Front) (net 1))
+  (segment (start 124.43 183.7875) (end 124.46 183.7575) (width 1) (layer Front) (net 2))
+  (segment (start 124.43 193.9225) (end 124.43 183.7875) (width 1) (layer Front) (net 2))
+  (segment (start 103.5725 183.8475) (end 103.46 183.96) (width 1) (layer Front) (net 3))
+  (segment (start 111.95 183.8475) (end 103.5725 183.8475) (width 1) (layer Front) (net 3))
+  (segment (start 111.95 189.696) (end 112.574 190.32) (width 1) (layer Front) (net 3))
+  (segment (start 111.95 183.8475) (end 111.95 189.696) (width 1) (layer Front) (net 3))
+  (segment (start 103.75 183.67) (end 103.46 183.96) (width 1) (layer Front) (net 3))
+  (segment (start 103.75 179) (end 103.75 183.67) (width 1) (layer Front) (net 3))
+  (segment (start 117.146 184.2915) (end 117.54 183.8975) (width 1) (layer Front) (net 4))
+  (segment (start 117.146 190.32) (end 117.146 184.2915) (width 1) (layer Front) (net 4))
+  (segment (start 110.735 196.92) (end 114.86 196.92) (width 1) (layer Front) (net 5))
+  (segment (start 99.3 196.92) (end 110.735 196.92) (width 1) (layer Front) (net 5))
+  (segment (start 93.08 190.7) (end 99.3 196.92) (width 1) (layer Front) (net 5))
+  (segment (start 93.08 188.65) (end 93.08 190.7) (width 1) (layer Front) (net 5))
+  (segment (start 93.08 188.65) (end 93.08 181.26) (width 1) (layer Front) (net 5))
+  (segment (start 114.8825 196.8975) (end 114.86 196.92) (width 1) (layer Front) (net 5))
+  (segment (start 124.43 196.8975) (end 114.8825 196.8975) (width 1) (layer Front) (net 5))
+  (segment (start 117.54 180.21) (end 117.53 180.2) (width 1) (layer Front) (net 6))
+  (segment (start 117.54 180.9225) (end 117.54 180.21) (width 1) (layer Front) (net 6))
+  (segment (start 117.53 180.2) (end 117.53 177.62) (width 1) (layer Front) (net 6))
+  (segment (start 116.72 176.81) (end 111.97 176.81) (width 1) (layer Front) (net 6))
+  (segment (start 117.53 177.62) (end 116.72 176.81) (width 1) (layer Front) (net 6))
+  (segment (start 112 180.9225) (end 111.95 180.8725) (width 1) (layer Front) (net 6))
+  (segment (start 117.54 180.9225) (end 112 180.9225) (width 1) (layer Front) (net 6))
 )
